Commit message: Changed Tire Parameters

File: description/robot_core.xacro (robot description, xacro)
@@ -6,6 +6,6 @@
     <xacro:property name="chassis_height" value="0.05"/>
     <xacro:property name="chassis_mass" value="1.0"/>
-    <xacro:property name="wheel_radius" value="0.017"/>
-    <xacro:property name="wheel_thickness" value="0.016"/>
+    <xacro:property name="wheel_radius" value="0.021"/>
+    <xacro:property name="wheel_thickness" value="0.019"/>
     <xacro:property name="wheel_mass" value="0.03"/>
     <xacro:property name="wheel_offset_x" value="-0.0"/>
@@ -85,8 +85,8 @@
         <collision>
             <geometry>
-                <cylinder radius="0.017" length="0.001" />
+                <cylinder radius="0.021" length="0.001" />
             </geometry>
         </collision>
-        <xacro:inertial_cylinder mass="0.1" length="0.02" radius="0.017">
+        <xacro:inertial_cylinder mass="0.1" length="0.02" radius="0.021">
         <origin xyz="0 0 0" rpy="0 0 0"/>
         </xacro:inertial_cylinder>
@@ -111,8 +111,8 @@
         <collision>
             <geometry>
-                <cylinder radius="0.017" length="0.001" />
+                <cylinder radius="0.021" length="0.001" />
             </geometry>
         </collision>
-        <xacro:inertial_cylinder mass="0.1" length="0.02" radius="0.017">
+        <xacro:inertial_cylinder mass="0.1" length="0.02" radius="0.021">
         <origin xyz="0 0 0" rpy="0 0 0"/>
         </xacro:inertial_cylinder>

File: description/ros2_control.xacro (robot description, xacro)
@@ -11,5 +11,5 @@
                 <param name="baud_rate">57600</param>
                 <param name="timeout">1000</param>
-                <param name="enc_counts_per_rev">480</param>
+                <param name="enc_counts_per_rev">1600</param>
             </hardware>
             <joint name="left_wheel_joint">
